Commit message: fix

File: robothon2022_description/urdf/robothon.xacro (robot description, xacro)
@@ -3,4 +3,10 @@
   <!-- Robothon cell -->
   <xacro:include filename="$(find robothon2022_description)/urdf/robothon_cell.urdf.xacro" />
+  <link name="world"/>
+  <joint name="world_to_table" type="fixed">
+    <parent link="world"/>
+    <child link="table"/>
+    <origin xyz="0 0 0"/>
+  </joint>
   <xacro:robothon_cell
     kinematics_parameters_file='$(find robothon2022_configurations)/config/calibration.yaml'

Commit message: boh

File: robothon2022_description/urdf/robothon.xacro (robot description, xacro)
@@ -11,4 +11,5 @@
   <xacro:robothon_cell
     kinematics_parameters_file='$(find robothon2022_configurations)/config/calibration.yaml'
+    joint_limits_parameters_file='$(find robothon2022_configurations)/config/joint_limits.yaml'
   /> <!--DO NOT DELETE -->
 </robot>

File: robothon2022_description/urdf/robothon_cell.urdf.xacro (robot description, xacro)
@@ -4,5 +4,5 @@
  "prefix:=''
   kinematics_parameters_file:='$(find ur_description)/config/ur3/default_kinematics.yaml'
-  joint_limits_parameters_file:='$(find ur_description)/config/ur3/joint_limits.yaml'
+  joint_limits_parameters_file:='$(find robothon2022_configurations)/config/joint_limits.yaml'
   physical_parameters_file:='$(find ur_description)/config/ur3/physical_parameters.yaml'
   transmission_hw_interface:=hardware_interface/PositionJointInterface
@@ -39,4 +39,5 @@
   <xacro:ur3_robotiq
     kinematics_parameters_file = "${kinematics_parameters_file}"
+    joint_limits_parameters_file = "${joint_limits_parameters_file}"
   />
   <link name="roof">
@@ -63,6 +64,13 @@
      <parent link="base_link"/>
      <child link="roof"/>
-     <origin xyz="0 0 0.65"/>
+     <origin xyz="0 -0.85 0.65"/>
    </joint>
+   <joint name="tool0_to_tip" type="fixed">
+     <parent link="tool0"/>
+     <child link="tip"/>
+     <origin xyz="0 0 0.157"/>
+   </joint>
+   <link name="tip">
+   </link>
 </xacro:macro>
 </robot>
