Commit message: ok and added frame

File: robothon2022_description/urdf/robothon_cell.urdf.xacro (robot description, xacro)
@@ -10,5 +10,5 @@
   safety_pos_margin:=0.15
   safety_k_position:=20 ">
-  <xacro:property name="grey" value="0.517647058823529	0.529411764705882	0.537254901960784 1" />
+  <xacro:property name="grey" value="0.517647058823529	0.529411764705882	0.537254901960784 0.3" />
   <link name="table">
      <visual>
@@ -31,9 +31,4 @@
      </collision>
    </link>
-   <!-- <joint name="world_to_robot" type="fixed">
-     <parent link="world"/>
-     <child link="base_link"/>
-     <origin xyz="0 0 0"/>
-   </joint> -->
    <joint name="table_to_robot" type="fixed">
      <parent link="table"/>
@@ -45,4 +40,29 @@
     kinematics_parameters_file = "${kinematics_parameters_file}"
   />
+  <link name="roof">
+     <visual>
+       <origin xyz="${0} ${0} ${0}" rpy="0 0 0" />
+       <geometry>
+         <box size="${2} ${2} ${0.15}" />
+       </geometry>
+       <material name="Grey">
+         <color rgba="${grey}"/>
+       </material>
+     </visual>
+     <collision>
+       <origin xyz="${0} ${0} ${0}" rpy="0 0 0" />
+       <geometry>
+         <box size="${2} ${2} ${0.15}" />
+       </geometry>
+       <material name="Grey">
+         <color rgba="${grey}"/>
+       </material>
+     </collision>
+   </link>
+   <joint name="robot_to_roof" type="fixed">
+     <parent link="base_link"/>
+     <child link="roof"/>
+     <origin xyz="0 0 0.65"/>
+   </joint>
 </xacro:macro>
 </robot>

Commit message: before change

File: robothon2022_description/urdf/robothon_cell.urdf.xacro (robot description, xacro)
@@ -31,4 +31,29 @@
      </collision>
    </link>
+   <link name="box">
+      <visual>
+        <origin xyz="${0} ${0} ${0}" rpy="0 0 0" />
+        <geometry>
+          <box size="${2} ${1} ${0.05}" />
+        </geometry>
+        <material name="Grey">
+          <color rgba="${grey}"/>
+        </material>
+      </visual>
+      <collision>
+        <origin xyz="${0} ${0} ${0}" rpy="0 0 0" />
+        <geometry>
+          <box size="${2} ${1} ${0.05}" />
+        </geometry>
+        <material name="Grey">
+          <color rgba="${grey}"/>
+        </material>
+      </collision>
+    </link>
+    <joint name="robot_to_box" type="fixed">
+      <parent link="base_link"/>
+      <child link="box"/>
+      <origin xyz="0.00 0.70 0.12"/>
+    </joint>
    <joint name="table_to_robot" type="fixed">
      <parent link="table"/>

Commit message: works

File: robothon2022_description/urdf/robothon_cell.urdf.xacro (robot description, xacro)
@@ -54,5 +54,5 @@
       <parent link="base_link"/>
       <child link="box"/>
-      <origin xyz="0.00 0.70 0.12"/>
+      <origin xyz="0.00 -0.70 0.12"/>
     </joint>
    <joint name="table_to_robot" type="fixed">
